File: LPF.sch (KiCad schematic (older format))
At the start: 124 parts, among them J1 Conn_02x05_Counter_Clockwise, P1 SMA, P3 SMA, P4 SMA

Commit message: added choke ferrite on each command line
Parts:
- added L17, L24, L25, L26, L27, L28, L29, L30, L31, L32, L33, L34, L35, L36, L37: Choke, Inductors_SMD:L_0805_HandSoldering, symbol L_Core_Ferrite_Small
- C69: value C -> 18p
Connections:
- net 12/10m: now also L29.2, L36.1; no longer C58.2, C6.1, D13.2 (A), D8.2 (A), RL14.16, RL7.1
- net 160m: now also L24.2, L31.1; no longer C1.1, C52.2, D2.2 (A), D3.2 (A), RL2.1, RL9.16
- net 17/15m: now also L28.2, L35.1; no longer C5.1, C57.2, D12.2 (A), D7.2 (A), RL13.16, RL6.1
- net 30/20m: now also L27.2, L34.1; no longer C4.1, C56.2, D11.2 (A), D6.2 (A), RL12.16, RL5.1
- net 40m: now also L26.2, L33.1; no longer C3.1, C54.2, D15.2 (A), D5.2 (A), RL11.16, RL4.1
- net 6m_Bypass: now also L30.2, L37.1; no longer C15.1, C70.2, D14.2 (A), D9.2 (A), RL15.16, RL8.1
- net 80m: now also L25.2, L32.1; no longer C2.1, C53.2, D10.2 (A), D4.2 (A), RL10.16, RL3.1
- net TX_RX_RLY: now also L17.2; no longer C7.1, D1.2 (A), RL1.16
- new net: C1.1, D3.2 (A), L24.1, RL2.1
- new net: C52.2, D2.2 (A), L31.2, RL9.16
- new net: C53.2, D10.2 (A), L32.2, RL10.16
- new net: C54.2, D15.2 (A), L33.2, RL11.16
- new net: C56.2, D11.2 (A), L34.2, RL12.16
- new net: C57.2, D12.2 (A), L35.2, RL13.16
- new net: C58.2, D13.2 (A), L36.2, RL14.16
- new net: C4.1, D6.2 (A), L27.1, RL5.1
- new net: C3.1, D5.2 (A), L26.1, RL4.1
- new net: C2.1, D4.2 (A), L25.1, RL3.1
- new net: C5.1, D7.2 (A), L28.1, RL6.1
- new net: C6.1, D8.2 (A), L29.1, RL7.1
- new net: C7.1, D1.2 (A), L17.1, RL1.16
- new net: C70.2, D14.2 (A), L37.2, RL15.16
- new net: C15.1, D9.2 (A), L30.1, RL8.1
Other:
- note removed: "IN"
- note removed: "Out"

Commit message: Caps changed for ATC-B footprint. Under dev., unstable
Parts:
- C11, C16, C17, C18, C19, C20, C21, C22, C23, C24, C25, C26, C27, C28, C29, C30, C31, C32, C33, C34, C35, C36, C37, C38, C39, C40, C41, C42, C43, C44, C45, C46, C47, C48, C49, C50, C51, C55, C59: footprint Capacitors_SMD:C_1210_HandSoldering -> ATC_B:ATC_500_HandSoldering
