File: LPF.kicad_pcb (KiCad board)
At the start: 4 copper layers, 100 x 100 mm, 587 parts, among them J1 Conn_02x05_Counter_Clockwise, P1 SMA, P2 SMA, P3 SMA, P4 SMA, P5 SMA, P6 SMA

Commit message: stitching errors corrected, new gerber
Parts:
- added REF**: via, via:via, F.Cu at (91.5, 139.0)
- added REF**: via, via:via, F.Cu at (93.5, 140.0)
- added REF**: via, via:via, F.Cu at (94.5, 140.0)
- added REF**: via, via:via, F.Cu at (95.5, 140.0)
- added REF**: via, via:via, F.Cu at (96.5, 140.0)
- added REF**: via, via:via, F.Cu at (97.5, 140.0)
- added REF**: via, via:via, F.Cu at (91.5, 141.0)
- added REF**: via, via:via, F.Cu at (92.5, 141.0)
- added REF**: via, via:via, F.Cu at (93.5, 141.0)
- added REF**: via, via:via, F.Cu at (94.5, 141.0)
- added REF**: via, via:via, F.Cu at (95.5, 141.0)
- added REF**: via, via:via, F.Cu at (92.5, 139.0)
- added REF**: via, via:via, F.Cu at (96.5, 141.0)
- added REF**: via, via:via, F.Cu at (97.5, 141.0)
- added REF**: via, via:via, F.Cu at (91.5, 142.0)
- added REF**: via, via:via, F.Cu at (92.5, 142.0)
- added REF**: via, via:via, F.Cu at (93.5, 142.0)
- added REF**: via, via:via, F.Cu at (94.5, 142.0)
- added REF**: via, via:via, F.Cu at (95.5, 142.0)
- added REF**: via, via:via, F.Cu at (96.5, 142.0)
- added REF**: via, via:via, F.Cu at (97.5, 142.0)
- added REF**: via, via:via, F.Cu at (91.5, 143.0)
- added REF**: via, via:via, F.Cu at (93.5, 139.0)
- added REF**: via, via:via, F.Cu at (92.5, 143.0)
- added REF**: via, via:via, F.Cu at (93.5, 143.0)
- added REF**: via, via:via, F.Cu at (94.5, 143.0)
- added REF**: via, via:via, F.Cu at (95.5, 143.0)
- added REF**: via, via:via, F.Cu at (96.5, 143.0)
- added REF**: via, via:via, F.Cu at (97.5, 143.0)
- added REF**: via, via:via, F.Cu at (91.5, 144.0)
- added REF**: via, via:via, F.Cu at (92.5, 144.0)
- added REF**: via, via:via, F.Cu at (93.5, 144.0)
- added REF**: via, via:via, F.Cu at (94.5, 144.0)
- added REF**: via, via:via, F.Cu at (94.5, 139.0)
- added REF**: via, via:via, F.Cu at (95.5, 144.0)
- added REF**: via, via:via, F.Cu at (96.5, 144.0)
- added REF**: via, via:via, F.Cu at (97.5, 144.0)
- added REF**: via, via:via, F.Cu at (95.5, 139.0)
- added REF**: via, via:via, F.Cu at (96.5, 139.0)
- added REF**: via, via:via, F.Cu at (97.5, 139.0)
- added REF**: via, via:via, F.Cu at (91.5, 140.0)
- added REF**: via, via:via, F.Cu at (92.5, 140.0)
Routing:
- net GND: track 1399.5 -> 1374.0 mm, vias 640 -> 649
