File: LPF.kicad_sch (KiCad schematic)
At the start: 138 parts, among them J1 Conn_02x05_Counter_Clockwise, P1 SMA, P3 SMA, P4 SMA

Commit message: minor changes, 1 bug fixed
Connections:
- net GND: no longer P3.1 (In), RL10.9, RL11.9, RL12.9, RL13.9, RL14.9, RL15.9, RL9.9
- net at RL12.8: now also P3.1 (In), RL10.8, RL10.9, RL11.8, RL11.9, RL12.9, RL13.8, RL13.9, RL14.8, RL14.9, RL15.8, RL15.9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
